Commit message: update

File: assets/RM_description/robot/robomaster.urdf (robot description, URDF)
Before this commit: robot robomaster_ep, 99 links, 98 joints
Joints:
- joint front_left_wheel_joint: limit effort=30 velocity=5 -> effort=30 velocity=10
- joint front_right_wheel_joint: limit effort=30 velocity=5 -> effort=30 velocity=10
- joint rear_left_wheel_joint: limit effort=30 velocity=5 -> effort=30 velocity=10
- joint rear_right_wheel_joint: limit effort=30 velocity=5 -> effort=30 velocity=10
